Commit message: adjust the URDF to the real machine

File: robots/uuv_d/robots/prototype_202605/robot.gazebo.xacro (robot description, xacro)
@@ -8,4 +8,21 @@
   <xacro:include filename="$(find aerial_robot_simulation)/xacro/spinal.gazebo.xacro" />
   <xacro:gazebo_spinal robot_name="$(arg robot_name)" gps_frame="fc"/>
+  <xacro:macro name="gazebo_link_color" params="link rgba emissive">
+    <gazebo reference="${link}">
+      <ambient>${rgba}</ambient>
+      <diffuse>${rgba}</diffuse>
+      <specular>0.3 0.3 0.3 1.0</specular>
+      <emissive>${emissive}</emissive>
+    </gazebo>
+  </xacro:macro>
+  <!-- Gazebo does not pick up the RViz-side material overrides for these meshes. -->
+  <xacro:gazebo_link_color link="t1" rgba="0.75 1.0 0.2 1.0" emissive="0.18 0.24 0.05 1.0"/>
+  <xacro:gazebo_link_color link="t2" rgba="0.75 1.0 0.2 1.0" emissive="0.18 0.24 0.05 1.0"/>
+  <xacro:gazebo_link_color link="t3" rgba="0.75 1.0 0.2 1.0" emissive="0.18 0.24 0.05 1.0"/>
+  <xacro:gazebo_link_color link="t4" rgba="0.75 1.0 0.2 1.0" emissive="0.18 0.24 0.05 1.0"/>
+  <xacro:gazebo_link_color link="t5" rgba="0.75 1.0 0.2 1.0" emissive="0.18 0.24 0.05 1.0"/>
+  <xacro:gazebo_link_color link="t6" rgba="0.75 1.0 0.2 1.0" emissive="0.18 0.24 0.05 1.0"/>
+  <xacro:gazebo_link_color link="t7" rgba="0.75 1.0 0.2 1.0" emissive="0.18 0.24 0.05 1.0"/>
+  <xacro:gazebo_link_color link="t8" rgba="0.75 1.0 0.2 1.0" emissive="0.18 0.24 0.05 1.0"/>
   <gazebo reference="root_joint">
     <disableFixedJointLumping>true</disableFixedJointLumping>
@@ -13,5 +30,5 @@
   <gazebo>
     <plugin name="uuv_plugin" filename="libuuv_underwater_object_ros_plugin.so">
-      <fluid_density>1000.0</fluid_density>
+      <fluid_density>0.002</fluid_density>
       <flow_velocity_topic>/hydrodynamics/current_velocity</flow_velocity_topic>
       <debug>1</debug>
@@ -19,6 +36,6 @@
         <neutrally_buoyant>0</neutrally_buoyant>
         <!-- todo: adjust the volume according to the real robot -->
-        <volume>0.001</volume>
-        <scaling_volume>0.0</scaling_volume>
+        <volume>1</volume>
+        <scaling_volume>1.0</scaling_volume>
         <box>
           <width>0.28</width>

File: robots/uuv_d/robots/prototype_202605/robot.urdf.xacro (robot description, xacro)
@@ -20,9 +20,9 @@
     <axis xyz="0 0 1"/>
   </joint>
-  <link name="base_link">
-    <inertial>
-      <origin xyz="-4.2558e-06 1.1226e-05 -0.2159" rpy="0.0 -0.0 0.0"/>
-      <mass value="1.9086"/>
-      <inertia ixx="0.016242" ixy="4.5627e-05" ixz="-4.7038e-11" iyy="0.016844" iyz="-1.7865e-11" izz="0.0050227"/>
+    <link name="base_link">
+    <inertial>
+      <origin xyz="-4.97441546509769e-06 1.31214560991818e-05 -0.165570321518981" rpy="0.0 -0.0 0.0"/>
+      <mass value="1.63288702957867"/>
+      <inertia ixx="0.0078532701523496" ixy="4.15087212249553e-05" ixz="-4.67638765406896e-11" iyy="0.00846439581729698" iyz="-1.77459249477566e-11" izz="0.00422885102236487"/>
     </inertial>
     <visual>
@@ -35,5 +35,5 @@
     <collision>
       <geometry>
-        <mesh filename="package://uuv_d/urdf/mesh/proto_type/meshes/base_link.STL"/>
+        <mesh filename="package://uuv_d/urdf/mesh/proto_type/meshes/base_link.stl"/>
       </geometry>
       <origin xyz="0.0 0.0 0.0" rpy="0.0 -0.0 0.0"/>
@@ -48,5 +48,5 @@
     <visual>
       <geometry>
-        <mesh filename="package://uuv_d/urdf/mesh/proto_type/meshes/t1.STL"/>
+        <mesh filename="package://uuv_d/urdf/mesh/proto_type/meshes/t1.dae"/>
       </geometry>
       <material name="__unnamed_material_2"/>
@@ -55,5 +55,5 @@
     <collision>
       <geometry>
-        <mesh filename="package://uuv_d/urdf/mesh/proto_type/meshes/t1.STL"/>
+        <mesh filename="package://uuv_d/urdf/mesh/proto_type/meshes/t1.stl"/>
       </geometry>
       <origin xyz="0.0 0.0 0.0" rpy="0.0 -0.0 0.0"/>
@@ -62,11 +62,11 @@
   <link name="thrust1">
     <inertial>
-      <origin xyz="0 0 0" rpy="0.0 0.0 0.0"/>
-      <mass value="0.00001"/>
-      <inertia ixx="0.00001" ixy="0.0" ixz="0.0" iyy="0.00001" iyz="0" izz="0.00001"/>
-    </inertial>
-    <visual>
-      <geometry>
-        <mesh filename="package://uuv_d/urdf/mesh/proto_type/meshes/thrust1.STL"/>
+      <origin xyz="-1.19904086659517e-14 -2.5729418595688e-14 -0.000999999999986234" rpy="0.0 -0.0 0.0"/>
+      <mass value="0.00283424938765199"/>
+      <inertia ixx="6.52506444943004e-07" ixy="-1.05879118406788e-21" ixz="3.04402465419514e-22" iyy="6.52506444942997e-07" iyz="-3.97046694025453e-22" izz="1.30312339029423e-06"/>
+    </inertial>
+    <visual>
+      <geometry>
+        <mesh filename="package://uuv_d/urdf/mesh/proto_type/meshes/thrust1.dae"/>
       </geometry>
       <material name="__unnamed_material_3"/>
@@ -75,5 +75,5 @@
     <collision>
       <geometry>
-        <mesh filename="package://uuv_d/urdf/mesh/proto_type/meshes/thrust1.STL"/>
+        <mesh filename="package://uuv_d/urdf/mesh/proto_type/meshes/thrust1.stl"/>
       </geometry>
       <origin xyz="0.0 0.0 0.0" rpy="0.0 -0.0 0.0"/>
@@ -82,4 +82,84 @@
   <link name="t2">
     <inertial>
+      <origin xyz="-0.0143 0.014292 0.017717" rpy="0.0 -0.0 0.0"/>
+      <mass value="0.099392"/>
+      <inertia ixx="7.9136e-05" ixy="-6.1395e-08" ixz="-3.804e-06" iyy="7.9154e-05" iyz="3.7817e-06" izz="7.672e-05"/>
+    </inertial>
+    <visual>
+      <geometry>
+        <mesh filename="package://uuv_d/urdf/mesh/proto_type/meshes/t2.dae"/>
+      </geometry>
+      <material name="__unnamed_material_4"/>
+      <origin xyz="0.0 0.0 0.0" rpy="0.0 -0.0 0.0"/>
+    </visual>
+    <collision>
+      <geometry>
+        <mesh filename="package://uuv_d/urdf/mesh/proto_type/meshes/t2.stl"/>
+      </geometry>
+      <origin xyz="0.0 0.0 0.0" rpy="0.0 -0.0 0.0"/>
+    </collision>
+  </link>
+  <link name="thrust2">
+    <inertial>
+      <origin xyz="1.13242748511766e-14 2.95874436062604e-14 0.00100000000002698" rpy="0.0 -0.0 0.0"/>
+      <mass value="0.00283424938765202"/>
+      <inertia ixx="6.52506444943003e-07" ixy="5.05572790392411e-21" ixz="5.69100261436483e-22" iyy="6.52506444943006e-07" iyz="-1.05879118406788e-22" izz="1.30312339029424e-06"/>
+    </inertial>
+    <visual>
+      <geometry>
+        <mesh filename="package://uuv_d/urdf/mesh/proto_type/meshes/thrust2.dae"/>
+      </geometry>
+      <material name="__unnamed_material_5"/>
+      <origin xyz="0.0 0.0 0.0" rpy="0.0 -0.0 0.0"/>
+    </visual>
+    <collision>
+      <geometry>
+        <mesh filename="package://uuv_d/urdf/mesh/proto_type/meshes/thrust2.stl"/>
+      </geometry>
+      <origin xyz="0.0 0.0 0.0" rpy="0.0 -0.0 0.0"/>
+    </collision>
+  </link>
+  <link name="t3">
+    <inertial>
+      <origin xyz="0.014292 0.0143 0.017717" rpy="0.0 -0.0 0.0"/>
+      <mass value="0.099392"/>
+      <inertia ixx="7.9154e-05" ixy="6.1395e-08" ixz="3.7817e-06" iyy="7.9136e-05" iyz="3.804e-06" izz="7.672e-05"/>
+    </inertial>
+    <visual>
+      <geometry>
+        <mesh filename="package://uuv_d/urdf/mesh/proto_type/meshes/t3.dae"/>
+      </geometry>
+      <material name="__unnamed_material_6"/>
+      <origin xyz="0.0 0.0 0.0" rpy="0.0 -0.0 0.0"/>
+    </visual>
+    <collision>
+      <geometry>
+        <mesh filename="package://uuv_d/urdf/mesh/proto_type/meshes/t3.stl"/>
+      </geometry>
+      <origin xyz="0.0 0.0 0.0" rpy="0.0 -0.0 0.0"/>
+    </collision>
+  </link>
+  <link name="thrust3">
+    <inertial>
+      <origin xyz="-1.62092561595273e-14 2.35644836976689e-14 0.00100000000001926" rpy="0.0 -0.0 0.0"/>
+      <mass value="0.002834249387652"/>
+      <inertia ixx="6.52506444942998e-07" ixy="4.18222517706811e-21" ixz="-6.61744490042422e-23" iyy="6.52506444943007e-07" iyz="-5.29395592033938e-23" izz="1.30312339029424e-06"/>
+    </inertial>
+    <visual>
+      <geometry>
+        <mesh filename="package://uuv_d/urdf/mesh/proto_type/meshes/thrust3.dae"/>
+      </geometry>
+      <material name="__unnamed_material_7"/>
+      <origin xyz="0.0 0.0 0.0" rpy="0.0 -0.0 0.0"/>
+    </visual>
+    <collision>
+      <geometry>
+        <mesh filename="package://uuv_d/urdf/mesh/proto_type/meshes/thrust3.stl"/>
+      </geometry>
+      <origin xyz="0.0 0.0 0.0" rpy="0.0 -0.0 0.0"/>
+    </collision>
+  </link>
+  <link name="t4">
+    <inertial>
       <origin xyz="0.0143 -0.014292 0.017717" rpy="0.0 -0.0 0.0"/>
       <mass value="0.099392"/>
@@ -88,85 +168,5 @@
     <visual>
       <geometry>
-        <mesh filename="package://uuv_d/urdf/mesh/proto_type/meshes/t2.STL"/>
-      </geometry>
-      <material name="__unnamed_material_4"/>
-      <origin xyz="0.0 0.0 0.0" rpy="0.0 -0.0 0.0"/>
-    </visual>
-    <collision>
-      <geometry>
-        <mesh filename="package://uuv_d/urdf/mesh/proto_type/meshes/t2.STL"/>
-      </geometry>
-      <origin xyz="0.0 0.0 0.0" rpy="0.0 -0.0 0.0"/>
-    </collision>
-  </link>
-  <link name="thrust2">
-    <inertial>
-      <origin xyz="0 0 0" rpy="0.0 0.0 0.0"/>
-      <mass value="0.00001"/>
-      <inertia ixx="0.00001" ixy="0.0" ixz="0.0" iyy="0.00001" iyz="0" izz="0.00001"/>
-    </inertial>
-    <visual>
-      <geometry>
-        <mesh filename="package://uuv_d/urdf/mesh/proto_type/meshes/thrust2.STL"/>
-      </geometry>
-      <material name="__unnamed_material_5"/>
-      <origin xyz="0.0 0.0 0.0" rpy="0.0 -0.0 0.0"/>
-    </visual>
-    <collision>
-      <geometry>
-        <mesh filename="package://uuv_d/urdf/mesh/proto_type/meshes/thrust2.STL"/>
-      </geometry>
-      <origin xyz="0.0 0.0 0.0" rpy="0.0 -0.0 0.0"/>
-    </collision>
-  </link>
-  <link name="t3">
-    <inertial>
-      <origin xyz="-0.0143 0.014292 0.017717" rpy="0.0 -0.0 0.0"/>
-      <mass value="0.099392"/>
-      <inertia ixx="7.9136e-05" ixy="-6.1395e-08" ixz="-3.804e-06" iyy="7.9154e-05" iyz="3.7817e-06" izz="7.672e-05"/>
-    </inertial>
-    <visual>
-      <geometry>
-        <mesh filename="package://uuv_d/urdf/mesh/proto_type/meshes/t3.STL"/>
-      </geometry>
-      <material name="__unnamed_material_6"/>
-      <origin xyz="0.0 0.0 0.0" rpy="0.0 -0.0 0.0"/>
-    </visual>
-    <collision>
-      <geometry>
-        <mesh filename="package://uuv_d/urdf/mesh/proto_type/meshes/t3.STL"/>
-      </geometry>
-      <origin xyz="0.0 0.0 0.0" rpy="0.0 -0.0 0.0"/>
-    </collision>
-  </link>
-  <link name="thrust3">
-    <inertial>
-      <origin xyz="0 0 0" rpy="0.0 0.0 0.0"/>
-      <mass value="0.00001"/>
-      <inertia ixx="0.00001" ixy="0.0" ixz="0.0" iyy="0.00001" iyz="0" izz="0.00001"/>
-    </inertial>
-    <visual>
-      <geometry>
-        <mesh filename="package://uuv_d/urdf/mesh/proto_type/meshes/thrust3.STL"/>
-      </geometry>
-      <material name="__unnamed_material_7"/>
-      <origin xyz="0.0 0.0 0.0" rpy="0.0 -0.0 0.0"/>
-    </visual>
-    <collision>
-      <geometry>
-        <mesh filename="package://uuv_d/urdf/mesh/proto_type/meshes/thrust3.STL"/>
-      </geometry>
-      <origin xyz="0.0 0.0 0.0" rpy="0.0 -0.0 0.0"/>
-    </collision>
-  </link>
-  <link name="t4">
-    <inertial>
-      <origin xyz="0.014292 0.0143 0.017717" rpy="0.0 -0.0 0.0"/>
-      <mass value="0.099392"/>
-      <inertia ixx="7.9154e-05" ixy="6.1395e-08" ixz="3.7817e-06" iyy="7.9136e-05" iyz="3.804e-06" izz="7.672e-05"/>
-    </inertial>
-    <visual>
-      <geometry>
-        <mesh filename="package://uuv_d/urdf/mesh/proto_type/meshes/t4.STL"/>
+        <mesh filename="package://uuv_d/urdf/mesh/proto_type/meshes/t4.dae"/>
       </geometry>
       <material name="__unnamed_material_8"/>
@@ -175,5 +175,5 @@
     <collision>
       <geometry>
-        <mesh filename="package://uuv_d/urdf/mesh/proto_type/meshes/t4.STL"/>
+        <mesh filename="package://uuv_d/urdf/mesh/proto_type/meshes/t4.stl"/>
       </geometry>
       <origin xyz="0.0 0.0 0.0" rpy="0.0 -0.0 0.0"/>
@@ -182,11 +182,11 @@
   <link name="thrust4">
     <inertial>
-      <origin xyz="0 0 0" rpy="0.0 0.0 0.0"/>
-      <mass value="0.00001"/>
-      <inertia ixx="0.00001" ixy="0.0" ixz="0.0" iyy="0.00001" iyz="0" izz="0.00001"/>
-    </inertial>
-    <visual>
-      <geometry>
-        <mesh filename="package://uuv_d/urdf/mesh/proto_type/meshes/thrust4.STL"/>
+      <origin xyz="2.66453525910038e-15 2.57155408078802e-14 0.000999999999986345" rpy="0.0 -0.0 0.0"/>
+      <mass value="0.00283424938765204"/>
+      <inertia ixx="6.52506444943016e-07" ixy="-6.89537758624204e-21" ixz="-1.05879118406788e-22" iyy="6.52506444943005e-07" iyz="1.05879118406788e-22" izz="1.30312339029425e-06"/>
+    </inertial>
+    <visual>
+      <geometry>
+        <mesh filename="package://uuv_d/urdf/mesh/proto_type/meshes/thrust4.dae"/>
       </geometry>
       <material name="__unnamed_material_9"/>
@@ -195,5 +195,5 @@
     <collision>
       <geometry>
-        <mesh filename="package://uuv_d/urdf/mesh/proto_type/meshes/thrust4.STL"/>
+        <mesh filename="package://uuv_d/urdf/mesh/proto_type/meshes/thrust4.stl"/>
       </geometry>
       <origin xyz="0.0 0.0 0.0" rpy="0.0 -0.0 0.0"/>
@@ -208,5 +208,5 @@
     <visual>
       <geometry>
-        <mesh filename="package://uuv_d/urdf/mesh/proto_type/meshes/t5.STL"/>
+        <mesh filename="package://uuv_d/urdf/mesh/proto_type/meshes/t5.dae"/>
       </geometry>
       <material name="__unnamed_material_10"/>
@@ -215,5 +215,5 @@
     <collision>
       <geometry>
-        <mesh filename="package://uuv_d/urdf/mesh/proto_type/meshes/t5.STL"/>
+        <mesh filename="package://uuv_d/urdf/mesh/proto_type/meshes/t5.stl"/>
       </geometry>
       <origin xyz="0.0 0.0 0.0" rpy="0.0 -0.0 0.0"/>
@@ -222,25 +222,38 @@
   <link name="thrust5">
     <inertial>
-      <origin xyz="0 0 0" rpy="0.0 0.0 0.0"/>
-      <mass value="0.00001"/>
-      <inertia ixx="0.00001" ixy="0.0" ixz="0.0" iyy="0.00001" iyz="0" izz="0.00001"/>
-    </inertial>
+      <origin xyz="-3.99680288865056e-15 -8.46545056276682e-16 0.000999999999998336" rpy="0.0 -0.0 0.0"/>
+      <mass value="0.002834249387652"/>
+      <inertia ixx="6.52506444943002e-07" ixy="-7.00125670464883e-21" ixz="-1.85288457211878e-22" iyy="6.52506444943005e-07" iyz="-1.58818677610181e-22" izz="1.30312339029424e-06"/>
+    </inertial>
+    <visual>
+      <geometry>
+        <mesh filename="package://uuv_d/urdf/mesh/proto_type/meshes/thrust5.dae"/>
+      </geometry>
+      <material name="__unnamed_material_11"/>
+      <origin xyz="0.0 0.0 0.0" rpy="0.0 -0.0 0.0"/>
+    </visual>
+    <collision>
+      <geometry>
+        <mesh filename="package://uuv_d/urdf/mesh/proto_type/meshes/thrust5.stl"/>
+      </geometry>
+      <origin xyz="0.0 0.0 0.0" rpy="0.0 -0.0 0.0"/>
+    </collision>
   </link>
   <link name="t6">
     <inertial>
-      <origin xyz="-0.0143000152087087 -0.0142922441739046 -0.0177167300533436" rpy="0.0 -0.0 0.0"/>
-      <mass value="0.0993924873705024"/>
-      <inertia ixx="7.91363117744376e-05" ixy="6.13947103617769e-08" ixz="3.80401853538391e-06" iyy="7.91541243411415e-05" iyz="3.78172056208575e-06" izz="7.67197078219357e-05"/>
-    </inertial>
-    <visual>
-      <geometry>
-        <mesh filename="package://uuv_d/urdf/mesh/proto_type/meshes/t6.STL"/>
-      </geometry>
-      <material name="__unnamed_material_11"/>
-      <origin xyz="0.0 0.0 0.0" rpy="0.0 -0.0 0.0"/>
-    </visual>
-    <collision>
-      <geometry>
-        <mesh filename="package://uuv_d/urdf/mesh/proto_type/meshes/t6.STL"/>
+      <origin xyz="0.0143 0.014292 -0.017717" rpy="0.0 -0.0 0.0"/>
+      <mass value="0.099392"/>
+      <inertia ixx="7.9136e-05" ixy="6.1395e-08" ixz="-3.804e-06" iyy="7.9154e-05" iyz="-3.7817e-06" izz="7.672e-05"/>
+    </inertial>
+    <visual>
+      <geometry>
+        <mesh filename="package://uuv_d/urdf/mesh/proto_type/meshes/t6.dae"/>
+      </geometry>
+      <material name="__unnamed_material_12"/>
+      <origin xyz="0.0 0.0 0.0" rpy="0.0 -0.0 0.0"/>
+    </visual>
+    <collision>
+      <geometry>
+        <mesh filename="package://uuv_d/urdf/mesh/proto_type/meshes/t6.stl"/>
       </geometry>
       <origin xyz="0.0 0.0 0.0" rpy="0.0 -0.0 0.0"/>
@@ -249,18 +262,18 @@
   <link name="thrust6">
     <inertial>
-      <origin xyz="0 0 0" rpy="0.0 0.0 0.0"/>
-      <mass value="0.00001"/>
-      <inertia ixx="0.00001" ixy="0.0" ixz="0.0" iyy="0.00001" iyz="0" izz="0.00001"/>
-    </inertial>
-    <visual>
-      <geometry>
-        <mesh filename="package://uuv_d/urdf/mesh/proto_type/meshes/thrust6.STL"/>
-      </geometry>
-      <material name="__unnamed_material_12"/>
-      <origin xyz="0.0 0.0 0.0" rpy="0.0 -0.0 0.0"/>
-    </visual>
-    <collision>
-      <geometry>
-        <mesh filename="package://uuv_d/urdf/mesh/proto_type/meshes/thrust6.STL"/>
+      <origin xyz="-1.99840144432528e-15 1.31838984174237e-15 0.00099999999999012" rpy="0.0 -0.0 0.0"/>
+      <mass value="0.00283424938765201"/>
+      <inertia ixx="6.52506444943003e-07" ixy="-5.9557004103818e-22" ixz="-1.98523347012727e-22" iyy="6.52506444942998e-07" iyz="1.05879118406788e-22" izz="1.30312339029423e-06"/>
+    </inertial>
+    <visual>
+      <geometry>
+        <mesh filename="package://uuv_d/urdf/mesh/proto_type/meshes/thrust6.dae"/>
+      </geometry>
+      <material name="__unnamed_material_13"/>
+      <origin xyz="0.0 0.0 0.0" rpy="0.0 -0.0 0.0"/>
+    </visual>
+    <collision>
+      <geometry>
+        <mesh filename="package://uuv_d/urdf/mesh/proto_type/meshes/thrust6.stl"/>
       </geometry>
       <origin xyz="0.0 0.0 0.0" rpy="0.0 -0.0 0.0"/>
@@ -269,18 +282,18 @@
   <link name="t7">
     <inertial>
-      <origin xyz="0.204997340751786 0.0143000152101347 -0.0177167300564932" rpy="0.0 -0.0 0.0"/>
-      <mass value="0.0993924873705016"/>
-      <inertia ixx="7.91541243411232e-05" ixy="-6.13947103569633e-08" ixz="3.78172056208173e-06" iyy="7.91363117744202e-05" iyz="-3.80401853537825e-06" izz="7.67197078219122e-05"/>
-    </inertial>
-    <visual>
-      <geometry>
-        <mesh filename="package://uuv_d/urdf/mesh/proto_type/meshes/t7.STL"/>
-      </geometry>
-      <material name="__unnamed_material_13"/>
-      <origin xyz="0.0 0.0 0.0" rpy="0.0 -0.0 0.0"/>
-    </visual>
-    <collision>
-      <geometry>
-        <mesh filename="package://uuv_d/urdf/mesh/proto_type/meshes/t7.STL"/>
+      <origin xyz="-0.014292 0.0143 -0.017717" rpy="0.0 -0.0 0.0"/>
+      <mass value="0.099392"/>
+      <inertia ixx="7.9154e-05" ixy="-6.1395e-08" ixz="3.7817e-06" iyy="7.9136e-05" iyz="-3.804e-06" izz="7.672e-05"/>
+    </inertial>
+    <visual>
+      <geometry>
+        <mesh filename="package://uuv_d/urdf/mesh/proto_type/meshes/t7.dae"/>
+      </geometry>
+      <material name="__unnamed_material_14"/>
+      <origin xyz="0.0 0.0 0.0" rpy="0.0 -0.0 0.0"/>
+    </visual>
+    <collision>
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
Commit message: adjust motor_info & buoyancy

File: robots/uuv_d/robots/prototype_202605/robot.gazebo.xacro (robot description, xacro)
@@ -30,5 +30,5 @@
   <gazebo>
     <plugin name="uuv_plugin" filename="libuuv_underwater_object_ros_plugin.so">
-      <fluid_density>0.002</fluid_density>
+      <fluid_density>1000</fluid_density>
       <flow_velocity_topic>/hydrodynamics/current_velocity</flow_velocity_topic>
       <debug>1</debug>
@@ -36,5 +36,5 @@
         <neutrally_buoyant>0</neutrally_buoyant>
         <!-- todo: adjust the volume according to the real robot -->
-        <volume>0.002</volume>
+        <volume>0.0038</volume>
         <scaling_volume>1.0</scaling_volume>
         <box>

File: robots/uuv_d/robots/prototype_202605/robot.urdf.xacro (robot description, xacro)
@@ -23,6 +23,11 @@
     <inertial>
       <origin xyz="-4.97441546509769e-06 1.31214560991818e-05 -0.165570321518981" rpy="0.0 -0.0 0.0"/>
-      <mass value="1.63288702957867"/>
-      <inertia ixx="0.0078532701523496" ixy="4.15087212249553e-05" ixz="-4.67638765406896e-11" iyy="0.00846439581729698" iyz="-1.77459249477566e-11" izz="0.00422885102236487"/>
+<mass value="2.8"/>
+<inertia ixx="0.013466428496435968"
+         ixy="7.117725680010082e-05"
+         ixz="-8.018855679667977e-11"
+         iyy="0.014514358837516688"
+         iyz="-3.042990050973674e-11"
+         izz="0.007251440331225416"/>
     </inertial>
     <visual>
