Commit message: add wrench visualization

File: robots/uuv_d/robots/prototype_202605/robot.gazebo.xacro (robot description, xacro)
@@ -36,5 +36,5 @@
         <neutrally_buoyant>0</neutrally_buoyant>
         <!-- todo: adjust the volume according to the real robot -->
-        <volume>0.0038</volume>
+        <volume>0.0037</volume>
         <scaling_volume>1.0</scaling_volume>
         <box>
@@ -43,5 +43,5 @@
           <height>0.072</height>
         </box>
-        <center_of_buoyancy>0 0 0</center_of_buoyancy>
+        <center_of_buoyancy>0.000610809453814865 0 -0.1655</center_of_buoyancy>
         <hydrodynamic_model>
           <type>fossen</type>

File: robots/uuv_d/robots/prototype_202605/robot.urdf.xacro (robot description, xacro)
@@ -22,5 +22,5 @@
     <link name="base_link">
     <inertial>
-      <origin xyz="0.000610809453814865 0.162582918364251 -0.165570321518981" rpy="0.0 -0.0 0.0"/>
+      <origin xyz="0.000610809453814865 0 -0.165570321518981" rpy="0.0 -0.0 0.0"/>
 <mass value="2.8"/>
 <inertia ixx="0.013466428496435968"
