Commit message: fix PID gaim

File: robots/uuv_d/robots/prototype_202605/robot.urdf.xacro (robot description, xacro)
@@ -22,5 +22,5 @@
     <link name="base_link">
     <inertial>
-      <origin xyz="-4.97441546509769e-06 1.31214560991818e-05 -0.165570321518981" rpy="0.0 -0.0 0.0"/>
+      <origin xyz="0.000610809453814865 0.162582918364251 -0.165570321518981" rpy="0.0 -0.0 0.0"/>
 <mass value="2.8"/>
 <inertia ixx="0.013466428496435968"
