Commit message: change the default pitch and roll, add parameters of pitch and roll

File: robots/uuv_d/urdf/mesh/proto_type/urdf/proto_type_5-dae.urdf (robot description, URDF)
Before this commit: robot proto_type, 19 links, 18 joints
Links:
- removed link root
- link base_link: mass 2.8 -> 2.03290862810658; geometry collision mesh filename=package://proto_type_5/meshes/base_link.stl; visual mesh filename=package://proto_type_5/meshes/base_link.dae
- link fc: geometry collision mesh filename=package://proto_type_5/meshes/fc.stl; visual mesh filename=package://proto_type_5/meshes/fc.dae
- link t1: mass 0.099392 -> 0.0993924873704976; geometry collision mesh filename=package://proto_type_5/meshes/t1.stl; visual mesh filename=package://proto_type_5/meshes/t1.dae
- link t2: mass 0.099392 -> 0.099392487370497; geometry collision mesh filename=package://proto_type_5/meshes/t2.stl; visual mesh filename=package://proto_type_5/meshes/t2.dae
- link t3: mass 0.099392 -> 0.099392487370502; geometry collision mesh filename=package://proto_type_5/meshes/t3.stl; visual mesh filename=package://proto_type_5/meshes/t3.dae
- link t4: mass 0.099392 -> 0.0993924873704986; geometry collision mesh filename=package://proto_type_5/meshes/t4.stl; visual mesh filename=package://proto_type_5/meshes/t4.dae
- link t5: mass 0.099392 -> 0.0993924873704979; geometry collision mesh filename=package://proto_type_5/meshes/t5.stl; visual mesh filename=package://proto_type_5/meshes/t5.dae
- link t6: mass 0.099392 -> 0.0993924873704977; geometry collision mesh filename=package://proto_type_5/meshes/t6.stl; visual mesh filename=package://proto_type_5/meshes/t6.dae
- link t7: mass 0.099392 -> 0.0993924873704991; geometry collision mesh filename=package://proto_type_5/meshes/t7.stl; visual mesh filename=package://proto_type_5/meshes/t7.dae
- link t8: mass 0.099392 -> 0.099392487370502; geometry collision mesh filename=package://proto_type_5/meshes/t8.stl; visual mesh filename=package://proto_type_5/meshes/t8.dae
- link thrust1: mass 0.00283424938765199 -> 0.0028342; geometry collision mesh filename=package://proto_type_5/meshes/thrust1.stl; visual mesh filename=package://proto_type_5/meshes/thrust1.dae
- link thrust2: mass 0.00283424938765202 -> 0.0028342; geometry collision mesh filename=package://proto_type_5/meshes/thrust2.stl; visual mesh filename=package://proto_type_5/meshes/thrust2.dae
- link thrust3: mass 0.002834249387652 -> 0.00283424938765202; geometry collision mesh filename=package://proto_type_5/meshes/thrust3.stl; visual mesh filename=package://proto_type_5/meshes/thrust3.dae
- link thrust4: mass 0.00283424938765204 -> 0.00283424938765201; geometry collision mesh filename=package://proto_type_5/meshes/thrust4.stl; visual mesh filename=package://proto_type_5/meshes/thrust4.dae
- link thrust5: mass 0.002834249387652 -> 0.00283424938765203; geometry collision mesh filename=package://proto_type_5/meshes/thrust5.stl; visual mesh filename=package://proto_type_5/meshes/thrust5.dae
- link thrust6: mass 0.00283424938765201 -> 0.00283424938765203; geometry collision mesh filename=package://proto_type_5/meshes/thrust6.stl; visual mesh filename=package://proto_type_5/meshes/thrust6.dae
- link thrust7: mass 0.002834249387652 -> 0.00283424938765203; geometry collision mesh filename=package://proto_type_5/meshes/thrust7.stl; visual mesh filename=package://proto_type_5/meshes/thrust7.dae
- link thrust8: mass 0.00283424938765202 -> 0.00283424938765205; geometry collision mesh filename=package://proto_type_5/meshes/thrust8.stl; visual mesh filename=package://proto_type_5/meshes/thrust8.dae
Joints:
- removed joint root_joint
- joint fc: origin xyz=0.0159087640700997 -0.0207051311296346 -0.13949999898 rpy=1.5707963267949 -0.0 1.93316031571781 -> xyz=0.00704662191902883 0.00267140409614365 -0.114499999725 rpy=0.0 -0.0 0.0
- joint l1: origin xyz=0.109644792463034 0.0969168704014227 -0.281585755800395 rpy=0.0 -0.0 0.0 -> xyz=0.109644792463 0.0969168704010846 -0.281585755800402 rpy=0.0 -0.0 0.0
- joint rotor1: limit lower=-30.0 upper=30.0 effort=100.0 velocity=0.5 -> effort=0.0 velocity=0.0
- joint rotor2: limit lower=-30.0 upper=30.0 effort=100.0 velocity=0.5 -> effort=0.0 velocity=0.0
- joint rotor3: limit lower=-30.0 upper=30.0 effort=100.0 velocity=0.5 -> effort=0.0 velocity=0.0
- joint rotor4: limit lower=-30.0 upper=30.0 effort=100.0 velocity=0.5 -> effort=0.0 velocity=0.0
- joint rotor5: limit lower=-30.0 upper=30.0 effort=100.0 velocity=0.5 -> effort=0.0 velocity=0.0
- joint rotor6: limit lower=-30.0 upper=30.0 effort=100.0 velocity=0.5 -> effort=0.0 velocity=0.0
- joint rotor7: limit lower=-30.0 upper=30.0 effort=100.0 velocity=0.5 -> effort=0.0 velocity=0.0
- joint rotor8: limit lower=-30.0 upper=30.0 effort=100.0 velocity=0.5 -> effort=0.0 velocity=0.0
